File: Schematic and PCB/charge_station.kicad_pcb (KiCad board)
At the start: 2 copper layers, 63 x 76 mm, 19 parts, among them J1 USB A module 3, J2 USB A module, J3 USB A module 2, J4 PAM8403 Bluetooth power, J5 Power supply, J6 TFT module, J7 strip led, Q1 BS250, Q2 BS250, U1 ESP32-DevKitC

Commit message: Add files via upload
Parts:
- moved U1 52.3 mm to (40.9, 56.7), turned to 0 degrees
- moved F2 8.75 mm to (92.5, 50.5)
- moved J1 8.75 mm to (91.8, 44.2)
- moved J2 7.50 mm to (91.5, 68.0)
- moved J6 7.15 mm to (72.2, 72.2), turned to 0 degrees
- moved F3 7.10 mm to (92.4, 74.9)
- moved F4 5.90 mm to (92.2, 99.7)
- moved J3 5.52 mm to (91.4, 92.5)
Routing:
- net Net-(D2-K): track 5.62 -> 77.3 mm
- net Net-(J6-Pin_4): track 75.9 -> 16.7 mm
- net Net-(Q2-G): track 19.7 -> 65.0 mm
- net Net-(J6-Pin_6): track 57.4 -> 20.1 mm
- net Net-(J6-Pin_3): track 47.7 -> 11.3 mm
- net Net-(J6-Pin_7): track 39.2 -> 6.01 mm
- net Net-(J1-Pin_4): track 263.6 -> 235.7 mm
- net Net-(J6-Pin_5): track 21.7 -> 40.8 mm
- net Net-(D1-K): track 210.9 -> 207.3 mm
- net Net-(J6-Pin_1): track 39.1 -> 37.3 mm
- net Net-(J3-Pin_1): track 10.3 -> 10.8 mm
- net Net-(J2-Pin_1): track 11.1 -> 10.6 mm
