File: Schematic and PCB/charge_station.kicad_sch (KiCad schematic)
At the start: 19 parts, among them J1 USB A module 3, J2 USB A module, J3 USB A module 2, J4 PAM8403 Bluetooth power, J5 Power supply, J6 TFT module, J7 strip led, Q1 BS250, Q2 BS250, U1 ESP32-DevKitC

Commit message: Add files via upload
Parts:
- removed F1: Fuse, Fuse:Fuse_Littelfuse_372_D8.50mm, symbol Device:Fuse
Connections:
- net at J5.1 (Pin_1): now also Q1.1 (D), Q1.2 (G)
Changed lines of the file:
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@@
 	(wire
 		(pts
-			(xy 43.18 74.93) (xy 46.99 74.93)
+			(xy 43.18 74.93) (xy 58.42 74.93)
 		)
 		(stroke
@@
 		(pts
 			(xy 257.81 49.53) (xy 240.03 49.53)
-		)
-		(stroke
-			(width 0)
-			(type default)
-		)
-	)
-	(wire
-		(pts
-			(xy 54.61 74.93) (xy 58.42 74.93)
 		)
 		(stroke
@@
 					(unit 1)
 				)
-			)
-		)
-	)
-	(symbol
-		(lib_id "Device:Fuse")
-		(at 50.8 74.93 90)
-		(unit 1)
-		(exclude_from_sim no)
-		(in_bom yes)
-		(on_board yes)
-		(dnp no)
-		(fields_autoplaced yes)
-		(property "Reference" "F1"
-			(at 50.8 68.58 90)
-			(effects
-				(font
-					(size 1.27 1.27)
-				)
-			)
-		)
-		(property "Value" "Fuse"
-			(at 50.8 71.12 90)
-			(effects
-				(font
-					(size 1.27 1.27)
-				)
-			)
-		)
-		(property "Footprint" "Fuse:Fuse_Littelfuse_372_D8.50mm"
-			(at 50.8 76.708 90)
-			(effects
-				(font
-					(size 1.27 1.27)
-				)
-				(hide yes)
-			)
-		)
-		(property "Datasheet" "~"
-			(at 50.8 74.93 0)
-			(effects
-				(font
-					(size 1.27 1.27)
-				)
-				(hide yes)
-			)
-		)
-		(property "Description" "Fuse"
-			(at 50.8 74.93 0)
-			(effects
-				(font
-					(size 1.27 1.27)
-				)
-				(hide yes)
-			)
-		)
-		(pin "1"
-		)
-		(pin "2"
-		)
-		(instances
-			(project ""
-				(path "/847a2b0c-685f-4b7a-9b79-7b59860b0dd8"
-					(reference "F1")
-					(unit 1)
-				)
